Commit message: Update scout_v2.urdf

File: scout_description/urdf/scout_v2.urdf (robot description, URDF)
Before this commit: robot scout_v2, 7 links, 6 joints
Links:
- link base_link: geometry collision box size=0.15416666666666667 0.627 0.06999999999999999; collision box size=0.925 0.38 0.21
- link front_left_wheel_link: geometry collision cylinder length=0.11653 radius=0.16459; visual mesh filename=file://$(find scout_description)/meshes/wheel_type2.dae
- link front_right_wheel_link: geometry collision cylinder length=0.11653 radius=0.16459; visual mesh filename=file://$(find scout_description)/meshes/wheel_type1.dae
- link rear_left_wheel_link: geometry collision cylinder length=0.11653 radius=0.16459; visual mesh filename=file://$(find scout_description)/meshes/wheel_type1.dae
- link rear_right_wheel_link: geometry collision cylinder length=0.11653 radius=0.16459; visual mesh filename=file://$(find scout_description)/meshes/wheel_type2.dae

Commit message: Update

File: scout_description/urdf/scout_v2.urdf (robot description, URDF)
Before this commit: robot scout_v2, 7 links, 6 joints
Links:
- link base_link: geometry collision box size=0.15416666666666667 0.627 0.06999999999999999; collision box size=0.925 0.38 0.21
- link front_left_wheel_link: geometry collision cylinder length=0.11653 radius=0.16459; visual mesh filename=package://scout_description/meshes/wheel_type2.dae
- link front_right_wheel_link: geometry collision cylinder length=0.11653 radius=0.16459; visual mesh filename=package://scout_description/meshes/wheel_type1.dae
- link rear_left_wheel_link: geometry collision cylinder length=0.11653 radius=0.16459; visual mesh filename=package://scout_description/meshes/wheel_type1.dae
- link rear_right_wheel_link: geometry collision cylinder length=0.11653 radius=0.16459; visual mesh filename=package://scout_description/meshes/wheel_type2.dae

Commit message: Update

File: scout_description/urdf/scout_v2.urdf (robot description, URDF)
Before this commit: robot scout_v2, 7 links, 6 joints
Joints:
- joint front_left_wheel: type fixed -> continuous
- joint front_right_wheel: type fixed -> continuous
- joint rear_left_wheel: type fixed -> continuous
- joint rear_right_wheel: type fixed -> continuous

File: scout_description/urdf/scout_v2.xacro (robot description, xacro)
@@ -75,7 +75,40 @@
             <plugin>gazebo_ros2_control/GazeboSystem</plugin>
         </hardware>
-        <joint name="scout_motor_fr_controller">
-            <command_interface name="position">
+        <!-- Wheel joints -->
+        <!-- Front Right Wheel Joint -->
+        <joint name="front_right_wheel">
+            <command_interface name="velocity">
+                <param name="min">-1</param>
+                <param name="max">1</param>
             </command_interface>
+            <state_interface name="position"/>
+            <state_interface name="velocity"/>
+        </joint>
+        <!-- Front Left Wheel Joint -->
+        <joint name="front_left_wheel">
+            <command_interface name="velocity">
+                <param name="min">-1</param>
+                <param name="max">1</param>
+            </command_interface>
+            <state_interface name="position"/>
+            <state_interface name="velocity"/>
+        </joint>
+        <!-- Rear Right Wheel Joint -->
+        <joint name="rear_right_wheel">
+            <command_interface name="velocity">
+                <param name="min">-1</param>
+                <param name="max">1</param>
+            </command_interface>
+            <state_interface name="position"/>
+            <state_interface name="velocity"/>
+        </joint>
+        <!-- Rear Left Wheel Joint -->
+        <joint name="rear_left_wheel">
+            <command_interface name="velocity">
+                <param name="min">-1</param>
+                <param name="max">1</param>
+            </command_interface>
+            <state_interface name="position"/>
+            <state_interface name="velocity"/>
         </joint>
     </ros2_control>
